File: kicad/lk201ps2/lk201ps2.kicad_pcb (KiCad board)
At the start: 2 copper layers, 50.8 x 50.8 mm, 17 parts, among them J1 RJ22, J2 Mini-DIN-6, U1 Itsy_Bitsy_5V, U2 ICL3232CPZ

Commit message: 1. Update board date.  This is board rev C 2. Bugfixes in scan software, fix a race condition between timing out keyboard data start and the arrival of the start bit.  This requires holding clock low long enough that any start is abandoned; if that is not done the byte may actually be sent if the interval between polls is short enough.
Other:
- board text added: "LK201 emulator by Paul Koning April 2021"
- board text removed: "LK201 emulator by Paul Koning March 2021"
